File: KiCad Files.kicad_sch (KiCad schematic)
At the start: 24 parts, among them SW1 SW_Push, U1 ATmega32U4-A, Y1 16MHz

Commit message: Final Changes to schematic
Made some final touches to the schematic before beginning the PCB
Connections:
- net +5V: no longer U1.24 (AVCC), U1.44 (AVCC)
- net COL0: no longer D1.1 (K), D2.1 (K), U1.27 (PD7)
- net GND: no longer U1.15 (GND), U1.23 (GND), U1.35 (GND), U1.43 (GND)
- new net: U1.15 (GND), U1.23 (GND), U1.35 (GND), U1.43 (GND)
- new net: U1.24 (AVCC), U1.44 (AVCC)
- new net ROW0: D1.1 (K), D2.1 (K), U1.27 (PD7)
Changed lines of the file:
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@@
   (junction (at 55.88 111.76) (diameter 0) (color 0 0 0 0)
   )
-  (junction (at 185.42 100.33) (diameter 0) (color 0 0 0 0)
-  )
   (junction (at 207.01 90.17) (diameter 0) (color 0 0 0 0)
-  )
-  (junction (at 88.9 43.18) (diameter 0) (color 0 0 0 0)
   )
   (junction (at 71.12 50.8) (diameter 0) (color 0 0 0 0)
@@
   )
   (junction (at 53.34 111.76) (diameter 0) (color 0 0 0 0)
-  )
-  (junction (at 86.36 134.62) (diameter 0) (color 0 0 0 0)
   )
   (junction (at 57.15 63.5) (diameter 0) (color 0 0 0 0)
@@
   )
   (wire (pts (xy 43.18 66.04) (xy 43.18 67.31))
-    (stroke (width 0) (type default))
-  )
-  (wire (pts (xy 86.36 134.62) (xy 88.9 134.62))
     (stroke (width 0) (type default))
   )
@@
     (stroke (width 0) (type default))
   )
-  (wire (pts (xy 177.8 100.33) (xy 185.42 100.33))
-    (stroke (width 0) (type default))
-  )
   (wire (pts (xy 43.18 54.61) (xy 43.18 62.23))
     (stroke (width 0) (type default))
@@
     (stroke (width 0) (type default))
   )
-  (wire (pts (xy 185.42 90.17) (xy 185.42 100.33))
-    (stroke (width 0) (type default))
-  )
   (wire (pts (xy 144.78 54.61) (xy 154.94 54.61))
     (stroke (width 0) (type default))
@@
     (stroke (width 0) (type default))
   )
-  (wire (pts (xy 185.42 100.33) (xy 199.39 100.33))
+  (wire (pts (xy 177.8 100.33) (xy 199.39 100.33))
     (stroke (width 0) (type default))
   )
@@
     (stroke (width 0) (type default))
   )
-  (wire (pts (xy 185.42 100.33) (xy 185.42 111.76))
+  (wire (pts (xy 185.42 90.17) (xy 185.42 111.76))
     (stroke (width 0) (type default))
   )
@@
     (stroke (width 0) (type default))
   )
-  (wire (pts (xy 88.9 43.18) (xy 91.44 43.18))
-    (stroke (width 0) (type default))
-  )
