File: KiCad Files.kicad_pcb (KiCad board)
At the start: 2 copper layers, 102.2 x 51.2 mm, 24 parts, among them SW1 SW_Push, U1 ATmega32U4-A, Y1 16MHz

Commit message: Finalized Tracing
Finished Optimizing tracing, and began running through errors.
Parts:
- added G***: LOGO, LOGO, B.Cu at (177.0, 83.1)
- D1, D2, D3, D4: moved to B.Cu
- moved SW1 6.61 mm to (143.5, 106.3)
- moved C7 5.98 mm to (134.4, 96.5), turned to -90 degrees
- moved R4 5.35 mm to (152.4, 100.9)
- moved C5 2.45 mm to (155.6, 87.3)
- turned R1 to -90 degrees
Connections:
- U1 pad 15: Net-(U1-GND-Pad15) -> GND
- U1 pad 23: Net-(U1-GND-Pad15) -> GND
- U1 pad 24: Net-(U1-AVCC-Pad24) -> +5V
- U1 pad 35: Net-(U1-GND-Pad15) -> GND
- U1 pad 43: Net-(U1-GND-Pad15) -> GND
- U1 pad 44: Net-(U1-AVCC-Pad24) -> +5V
Routing:
- net GND: track 77.1 -> 130.4 mm, vias 1 -> 2
- net Net-(U1-GND-Pad15): track 28.7 -> 0.00 mm
- net COL1: track 80.8 -> 108.8 mm, vias 4 -> 0
- net +5V: track 75.5 -> 100.9 mm, vias 2 -> 5
- net Net-(U1-AVCC-Pad24): track 19.5 -> 0.00 mm, vias 2 -> 0
- net unconnected-(USB1-SHIELD-Pad6): track 0.00 -> 16.3 mm
- net ROW1: track 55.0 -> 69.8 mm, vias 3 -> 0
- net Net-(U1-XTAL2): track 0.00 -> 11.2 mm
- net COL0: track 86.4 -> 97.3 mm, vias 4 -> 0
- net Net-(U1-XTAL1): track 0.00 -> 8.65 mm
- net Net-(U1-~{HWB}/PE2): track 0.00 -> 7.80 mm
- net Net-(U1-UCAP): track 0.00 -> 5.23 mm
- net Net-(U1-~{RESET}): track 42.4 -> 46.5 mm, vias 0 -> 2
- net Net-(U1-D+): track 17.4 -> 20.7 mm
- net ROW0: track 69.4 -> 71.8 mm, vias 1 -> 2
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- added copper zone on B.Cu, net GND
Other:
- board text added: "11/7/2023"
- board text added: "BapPad Prototype 1.0"
